File: usb-rj45-serial.sch (KiCad schematic (older format))
At the start: 11 parts

Commit message: Add TTL header
Parts:
- removed SW? (x2): Switch_SPDT_x2, symbol Switch_SPDT_x2
- added P2: TTL_Breakout, symbol CONN_01X06
- added SW1: V_Select, symbol DPDT
- added SW3: TTL_Sel, symbol DPDT
- C1, C2, C3, C4, C5: renamed from C?; value C_Small -> 100nF
- P1: renamed from P?; value CONN_01X06 -> CP2102_BOB
- SW2: renamed from SW?; value DPDT -> Rollover
- gave numbers to parts that had none: 2
Connections:
- net labels added: DTR_TTL, GND, RX_TTL, TX_TTL, VCC
- net labels removed: GNDREF, RX_OUT_TTL, TX_IN_TTL
- wire segments 39 -> 61
- no-connect marks 6 -> 12
Other:
- note added: "P1: CP2102 micro USB breakout board header"
- note added: "P2: Arduino Pro Mini pinout"
- note added: "SW1: 3.3/5V select switch"
- note added: "SW2: Rollover (null modem) switch for RJ45"
- note added: "SW3: Select RJ45/RS232 or TTL signal output"
- moved on the sheet: P1
